File: IRIS-core/IRIS-core.kicad_pcb (KiCad board)
At the start: 2 copper layers, 65 x 65 mm, 57 parts, among them J1 Conn_01x20_MountingPin, J2 SiPM, SW1 SW_Push, U1 Teensy4.1, U10 CAM-M8, U2 ST_Motion_Breakout, U3 LT1807, U4 MT25QL01GBBB8ESF-0SIT, U5 EVAL-ADXL372Z, U6 HSCDRRN001BDSA3, U7 TPD4E1U06, U8 TPD4E1U06, U9 TPD4E1U06

Commit message: Added BOM, IRIS core ready for review
Parts:
- C4: footprint Capacitor_SMD:C_0603_1608Metric -> Capacitor_SMD:C_0805_2012Metric
- J1: footprint star-common-lib:IRIS_Muons_Middle -> star-common-lib:IRIS_Muons_physical
- moved R1 31.8 mm to (19.2, -11.2), turned to 90 degrees
- moved R2 28.8 mm to (21.2, -11.2), turned to 90 degrees
- moved R13 9.50 mm to (41.8, 23.5)
- moved JP3 0.75 mm to (36.2, -12.0)
- moved R14 0.56 mm to (53.5, 26.2), turned to 0 degrees
- moved D2 0.25 mm to (29.2, 0.00)
- moved R12 0.25 mm to (11.5, 7.00)
Connections:
- net Net-(J1-Pad14) renamed /BCK_ALT
- J1 pad 3: /~PWR_BRD_INT -> /IO2
- J1 pad 7: /IO6 -> /~PWR_BRD_INT
- U1 pad 26: /HG_INT2 -> Net-(U1-Pad26)
- U1 pad 27: /HG_INT1 -> /HG_INT2
- U1 pad 28: Net-(U1-Pad28) -> /HG_INT1
- U1 pad 45: /GPS_INT -> Net-(U1-Pad45)
- U1 pad 5: /~PWR_BRD_INT -> /IO2
- U1 pad 9: /IO6 -> /~PWR_BRD_INT
- U10 pad 7: /GPS_INT -> Net-(U10-Pad7)
- U7 pad 3: /~PWR_BRD_INT -> /IO2
- U8 pad 3: /IO6 -> /~PWR_BRD_INT
- U9 pad 3: /MOSI_1 -> Net-(U9-Pad3)
- U9 pad 6: Net-(U9-Pad6) -> /MOSI_1
Routing:
- net /GPS_INT: track 33.6 -> 0.00 mm, vias 2 -> 0
- net +3V3: track 202.3 -> 220.5 mm
- net /IO6: track 9.16 -> 0.00 mm
- net /IO2: track 0.00 -> 9.16 mm
- net /~CS_HG: track 19.2 -> 27.9 mm, vias 1 -> 2
- net /FB_HV_N: track 57.4 -> 64.1 mm
- net /SiPM: track 2.11 -> 7.42 mm
- net Net-(C1-Pad1): track 25.2 -> 20.3 mm
- net /HG_INT2: track 28.9 -> 24.1 mm
- net /HG_INT1: track 28.4 -> 24.1 mm
- net /SCLK_1: track 75.5 -> 78.5 mm, vias 1 -> 0
- net +29.5V: track 60.8 -> 57.9 mm
- net /MISO_1: track 75.9 -> 73.8 mm, vias 1 -> 0
- net /on_off: track 56.6 -> 54.8 mm, vias 0 -> 2
- net /SCL_0: track 58.7 -> 56.9 mm
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Other:
- net class Default: via_dia 0.5588 -> 0.6; via_drill 0.254 -> 0.3
- rule via_min_drill: 0.2 -> 0.3
- rule via_min_size: 0.5588 -> 0.6
- board text added: "DNP if U10 Populated"
- board text removed: "DNP if U10 populated"
