File: IRIS-core/IRIS-core.sch (KiCad schematic (older format))
At the start: 18 parts

Commit message: IRIS Core V4.0 draft
Parts:
- removed C?: 0.1uF, symbol Device:C
- removed C? (x2): 47pF, symbol Device:C
- removed J?: USB_C_Receptacle_USB2.0, symbol Connector:USB_C_Receptacle_USB2.0
- removed Q? (x2): MBT3904DW1, Package_TO_SOT_SMD:SOT-363_SC-70-6, symbol Transistor_BJT:MBT3904DW1
- removed R? (x5): R, symbol Device:R
- removed R? (x2): 5.1k, symbol Device:R
- removed R? (x2): 10k, symbol Device:R
- removed U?: ESP32-WROVER, symbol esp32-wrover:ESP32-WROVER
- removed U?: FT231XS, Package_SO:SSOP-20_3.9x8.7mm_P0.635mm, symbol Interface_USB:FT231XS
- removed U?: TPD2E2U06, Package_TO_SOT_SMD:SOT-543, symbol Power_Protection:TPD2E2U06
- added BT1: CR1220 - Keystone 500, star-common-lib:CR12XX-Keystone-500, symbol Device:Battery_Cell
- added C1: 10pF, Capacitor_SMD:C_0603_1608Metric, symbol Device:C
- added C2, C6, C7, C8: 0.1uF, Capacitor_SMD:C_0603_1608Metric, symbol Device:C
- added C3: 10uF, Capacitor_SMD:C_0603_1608Metric, symbol Device:C
- added C4: 20nF, Capacitor_SMD:C_0603_1608Metric, symbol Device:C
- added C5: 0R, Capacitor_SMD:C_0603_1608Metric, symbol Device:C
- added C9: 1uF, Capacitor_SMD:C_0603_1608Metric, symbol Device:C
- added D1, D2: MBR0540, Diode_SMD:D_SOD-123, symbol Diode:MBR0540
- added D3: 150080RS75000, LED_SMD:LED_0805_2012Metric_Pad1.15x1.40mm_HandSolder, symbol Device:LED
- added D4: 150080VS75000, LED_SMD:LED_0805_2012Metric_Pad1.15x1.40mm_HandSolder, symbol Device:LED
- added D5: 150080YS75000, LED_SMD:LED_0805_2012Metric_Pad1.15x1.40mm_HandSolder, symbol Device:LED
- added FB1: 600, Inductor_SMD:L_0603_1608Metric, symbol Device:Ferrite_Bead
- added J1: Conn_01x20_MountingPin, star-common-lib:IRIS_Muons_Middle, symbol Connector_Generic_MountingPin:Conn_01x20_MountingPin
- added J2: SiPM, star-common-lib:SiPM, symbol Connector_Generic:Conn_02x03_Odd_Even
- added JP1, JP3: SolderJumper_2_Open, Jumper:SolderJumper-2_P1.3mm_Open_RoundedPad1.0x1.5mm, symbol Jumper:SolderJumper_2_Open
- added JP2: Write_Protect, Connector_PinHeader_2.54mm:PinHeader_1x02_P2.54mm_Horizontal, symbol Device:Jumper
- added NT1, NT2: Net-Tie_2, NetTie:NetTie-2_SMD_Pad0.5mm, symbol Device:Net-Tie_2
- added R1, R11, R12, R13, R14, R2, R5, R6: 10k, Resistor_SMD:R_0603_1608Metric, symbol Device:R
- added R10, R20, R21: 0R, Resistor_SMD:R_0603_1608Metric, symbol Device:R
- added R15, R16, R17: 100R, Resistor_SMD:R_0603_1608Metric, symbol Device:R
- added R18, R19: DNP, Resistor_SMD:R_0603_1608Metric, symbol Device:R
- added R3: 1k, Resistor_SMD:R_0603_1608Metric, symbol Device:R
- added R4: 249R, Resistor_SMD:R_0603_1608Metric, symbol Device:R
- added R7, R8: 100k, Resistor_SMD:R_0603_1608Metric, symbol Device:R
- added R9: 24.9k, Resistor_SMD:R_0603_1608Metric, symbol Device:R
- added SW1: SW_Push, Button_Switch_THT:SW_Tactile_SPST_Angled_PTS645Vx39-2LFS, symbol Switch:SW_Push
- added TP1: Raw, TestPoint:TestPoint_Keystone_5005-5009_Compact, symbol Connector:TestPoint_Probe
- added TP2: Amplified, TestPoint:TestPoint_Keystone_5005-5009_Compact, symbol Connector:TestPoint_Probe
- added U1: Teensy4.1, star-common-lib:Teensy41, symbol star-common-lib:Teensy4.1
- added U10: CAM-M8, star-common-lib:UBLOX_CAM_M8, symbol star-common-lib:CAM-M8
- added U2: ST_Motion_Breakout, star-common-lib:ST_Motion_Breakout, symbol star-common-lib:ST_Motion_Breakout
- added U3: LT1807, Package_SO:SOIC-8_3.9x4.9mm_P1.27mm, symbol star-common-lib:LT1807
- added U4: MT25QL01GBBB8ESF-0SIT, Package_SO:SOIC-16W_7.5x10.3mm_P1.27mm, symbol star-common-lib:MT25QL01GBBB8ESF-0SIT
- added U5: EVAL-ADXL372Z, star-common-lib:EVAL-ADXL372Z, symbol star-common-lib:EVAL-ADXL372Z
- added U6: HSCDRRN001BDSA3, star-common-lib:HSCDRRN001BDSA3, symbol star-common-lib:HSCDRRN001BDSA3
- added U7, U8, U9: TPD4E1U06, Package_TO_SOT_SMD:SOT-23-6, symbol star-common-lib:TPD4E1U06
Connections:
- net +3V3: now also C2.1, C3.1, C6.1, C7.1, C8.1, C9.1, R1.1, R11.1, R12.1, R13.1, R14.1, R15.2, R16.2, R17.2, R2.1, U1.15 (3V3), U1.46 (3V3), U1.51 (3V3), U10.1 (VCC_IO), U10.9 (VCC), U2.2 (3.3V), U3.8 (V+), U4.2 (Vcc), U5.1 (3.3V), U5.2 (VDDIO), U6.2 (3.3V)
- net GND: now also BT1.2 (-), C2.2, C3.2, C6.2, C7.2, C8.2, C9.2, FB1.2, J1.1 (Pin_1), J1.13 (Pin_13), J1.19 (Pin_19), J1.20 (Pin_20), J1.MP (MountPin), JP2.1, SW1.1, U1.1 (GND), U1.34 (GND), U1.47 (GND), U1.52 (GND), U10.10 (GND), U10.11 (GND), U10.12 (GND), U10.13 (GND), U10.14 (GND), U10.15 (GND), U10.18 (GND), U10.19 (GND), U10.21 (GND), U10.22 (GND), U10.27 (GND), U10.31 (GND), U10.4 (GND), U10.5 (GND), U2.1 (GND), U4.10 (Vss), U5.10 (GND), U5.3 (GND), U6.1 (GND), U7.2 (GND), U8.2 (GND), U9.2 (GND)
- new net: BT1.1 (+), JP3.1 (A)
- new net: J1.14 (Pin_14), JP1.1 (A)
- new net: U10.16 (RF_OUT), U10.17 (RF_IN)
- new net: R18.1, U10.25 (TXD/SPI_MISO)
- new net: R19.1, U10.26 (RXD/SPI_MOSI)
- new net: R20.1, U10.3 (SDA/SPI_CS)
- new net: R21.1, U10.6 (SCL/SPI_CLK)
- new net: C1.1, R5.1, R6.1, TP2.1, U3.1, U3.5 (+)
- new net: R3.1, TP1.1, U3.3 (+)
- new net: D3.2 (A), R15.1
- new net: D4.2 (A), R16.1
- new net: D5.2 (A), R17.1
- new net: C1.2, R4.1, R5.2, U3.2 (-)
- new net: D1.2 (A), R7.1, R8.2, U3.6 (-)
- new net: D1.1 (K), D2.2 (A), U3.7
- new net: C4.1, C5.2, D2.1 (K), R8.1
- new net: C5.1, R10.1, R9.2
- new net +29.5V: J1.18 (Pin_18), J2.2 (Pin_2), NT1.2
- new net +5V: J1.15 (Pin_15), U1.48 (VIN)
- new net Detector: R10.2, U1.36 (14_A0_TX3_SPDIF_OUT)
- new net FB_HV_N: J1.17 (Pin_17), J2.3 (Pin_3), NT2.1
- new net FB_HV_P: J1.16 (Pin_16), J2.1 (Pin_1), NT1.1
- new net GNDA: C4.2, FB1.1, J2.4 (Pin_4), NT2.2, R4.2, R6.2, R7.2, R9.1, U3.4 (V-)
- new net GPS_INT: U1.45 (23_A9_CRX1_MCLK1), U10.7 (EXTINT)
- new net HG_INT1: U1.27 (35_TX8), U5.5 (INT1)
- new net HG_INT2: U1.26 (34_RX8), U5.4 (INT2)
- new net IO1_SYNC: J1.2 (Pin_2), U1.4 (2_OUT2), U7.1 (IO1)
- new net IO3: J1.4 (Pin_4), U1.6 (4_BCLK2), U7.4 (IO3)
- new net IO4: J1.5 (Pin_5), U1.7 (5_IN2), U7.6 (IO4)
- new net IO5: J1.6 (Pin_6), U1.8 (6_OUT1D), U8.1 (IO1)
- new net IO6: J1.7 (Pin_7), U1.9 (7_RX2_OUT1A), U8.3 (IO2)
- new net MISO_0: U1.14 (12_MISO_MQSL), U4.8 (DQ1_(MISO))
- new net MISO_1: J1.10 (Pin_10), U1.31 (39_MISO1_OUT1A), U5.7 (MISO), U6.3 (MISO), U9.1 (IO1)
- new net MOSI_0: U1.13 (11_MOSI_CTX1), U4.15 (DQ0_(MOSI))
- new net MOSI_1: J1.11 (Pin_11), U1.18 (26_A12_MOSI1), U5.8 (MOSI), U9.3 (IO2)
- new net M_INT1: U1.16 (24_A10_TX6_SCL2), U2.6 (INT1)
- new net M_INT2: U1.33 (41_A17), U2.7 (INT2)
- new net M_INT3: U1.17 (25_A11_RX6_SDA2), U2.8 (INT3)
- new net M_INT4: U1.32 (40_A16), U2.9 (INT4)
- new net M_Wake: U1.37 (15_A1_RX3_SPDIF_IN), U2.3 (Wake)
- new net RGB_G: D4.1 (K), U1.24 (32_OUT1B)
- new net RGB_R: D3.1 (K), U1.22 (30_CRX3)
- new net RGB_Y: D5.1 (K), U1.23 (31_CTX3)
- new net RX_MCU: R18.2, U1.43 (21_A7_RX5_BCLK1)
- new net SCLK_0: U1.35 (13_SCK_LED), U4.16 (SCLK)
- new net SCLK_1: J1.12 (Pin_12), U1.19 (27_A13_SCK1), U5.9 (SCLK), U6.4 (SCLK), U9.4 (IO3)
- new net SCL_0: J1.9 (Pin_9), R1.2, R21.2, U1.41 (19_A5_SCL), U8.6 (IO4)
- new net SCL_1: U1.38 (16_A2_RX4_SCL1), U2.4 (SCL)
- new net SDA_0: J1.8 (Pin_8), R2.2, R20.2, U1.40 (18_A4_SDA), U8.4 (IO3)
- new net SDA_1: U1.39 (17_A3_TX4_SDA1), U2.5 (SDA)
- new net SiPM: J2.5 (Pin_5), J2.6 (Pin_6), R3.2
- new net TX_MCU: R19.2, U1.42 (20_A6_TX5_LRCLK1)
- new net VCC: JP1.2 (B), JP3.2 (B), U1.50 (VBAT), U10.8 (V_BCKP)
- new net on_off: SW1.2, U1.54 (ON_OFF)
- new net ~CS_HG: R13.2, U1.30 (38_CS1_IN1), U5.6 (CS)
- new net ~CS_MEM: U1.12 (10_CS_MQSR), U4.7 (~CS)
- new net ~CS_PITOT: R14.2, U1.25 (33_MCLK2), U6.5 (~CS)
- new net ~HOLD: R11.2, U4.1 (~HOLD(DQ3))
- new net ~PWR_BRD_INT: J1.3 (Pin_3), U1.5 (3_LRCLK2), U7.3 (IO2)
- new net ~RST_MEM: U1.11 (9_OUT1C), U4.3 (~RESET)
- new net ~WP: JP2.2, R12.2, U4.9 (~WP(DQ2))
- no-connect marks 10 -> 15
Other:
- note added: "512Mb (64MB) SPI Flash"
- note added: "All jumpers are remove\nbefore flight"
- note added: "CUT VUSB TRACE ON \nUNDERSIDE OF TEENSY"
- note added: "DNP if using \nGPS"
- note added: "Digital High-G Accelerometer"
- note added: "Primary Sensors"
- note added: "RGB Debug LED"
- note added: "SiPM Processing"

Commit message: Added BOM, IRIS core ready for review
Parts:
- BT1: Digikey P/N (none) -> 36-500-ND
- C1: Digikey P/N (none) -> 1276-1069-1-ND
- C2, C6, C7, C8: Digikey P/N (none) -> 1276-CL10B104KB8NNNLCT-ND
- C3: Digikey P/N (none) -> 1276-1192-1-ND
- C4: footprint Capacitor_SMD:C_0603_1608Metric -> Capacitor_SMD:C_0805_2012Metric; Digikey P/N (none) -> 478-10428-1-ND
- C5, R10, R20, R21: Digikey P/N (none) -> RMCF0603ZT0R00CT-ND
- C9: Digikey P/N (none) -> 1276-1102-1-ND
- D1, D2: Digikey P/N (none) -> MBR0540T3GOSCT-ND
- D3: Digikey P/N (none) -> 732-4984-1-ND
- D4: Digikey P/N (none) -> 732-4986-1-ND
- D5: Digikey P/N (none) -> 732-4987-1-ND
- FB1: Digikey P/N (none) -> 732-1593-1-ND
- J1: footprint star-common-lib:IRIS_Muons_Middle -> star-common-lib:IRIS_Muons_physical
- JP2: Digikey P/N (none) -> 2057-PH1RB-02-UA-ND
- R1, R11, R12, R13, R14, R2, R5, R6: Digikey P/N (none) -> RNCP0603FTD10K0CT-ND
- R15, R16, R17: Digikey P/N (none) -> RMCF0603FT100RCT-ND
- R3: Digikey P/N (none) -> RMCF0603FT1K00CT-ND
- R4: Digikey P/N (none) -> P249BLCT-ND
- R7, R8: Digikey P/N (none) -> RR08P100KDCT-ND
- R9: Digikey P/N (none) -> RR08P24.9KDCT-ND
- SW1: Digikey P/N (none) -> CKN9103-ND
- TP1, TP2: Digikey P/N (none) -> 36-5006-ND
- U10: Digikey P/N (none) -> 672-CAM-M8Q-0TR-ND
- U3: Digikey P/N (none) -> LT1807IS8#TRPBFCT-ND
- U4: Digikey P/N (none) -> 557-1789-ND
- U5: Digikey P/N (none) -> 1127-3597-ND
- U7, U8, U9: Digikey P/N (none) -> 296-35965-1-ND
Connections:
- net IO6 is gone; now on net ~PWR_BRD_INT: J1.7 (Pin_7), U1.9 (7_RX2_OUT1A), U8.3 (IO2)
- net HG_INT1: now also U1.28 (36_CS); no longer U1.27 (35_TX8)
- net HG_INT2: now also U1.27 (35_TX8); no longer U1.26 (34_RX8)
- net MOSI_1: now also U9.6 (IO4); no longer U9.3 (IO2)
- net ~PWR_BRD_INT: no longer J1.3 (Pin_3), U1.5 (3_LRCLK2), U7.3 (IO2)
- net BCK_ALT: now reaches J1.14 (Pin_14), JP1.1 (A)
- net GPS_INT: no longer names the net of U1.45 (23_A9_CRX1_MCLK1)
- net GPS_INT: no longer U10.7 (EXTINT)
- new net IO2: J1.3 (Pin_3), U1.5 (3_LRCLK2), U7.3 (IO2)
- no-connect marks 15 -> 17
Other:
- note added: "Differential Pressure Sensor"
- note added: "ESD Protection"
- note added: "GNSS Module (Optional)"
- note added: "IMU/Primary Sensors"
- note added: "Jumpers"
- note added: "Muons Amplifier and Peak Detector"
- note added: "Muons Detector Board Connector"
- note added: "On/Off Switch"
- note added: "Stack Connector"
- note added: "Teensy 4.1"
- note added: "Write Protect Jumper"
- note removed: "Primary Sensors"
- moved on the sheet: BT1, C1, C2, C3, C4, C5, C6, C7, C8, C9, D1, D2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
